File: 5way_cv_switch.kicad_pcb (KiCad board)
At the start: 2 copper layers, 29 x 22 mm, 20 parts, among them J1 I/O connector, J2 5-way Switch Connector, U1 HT7550-1, U2 LMV321IDBVR

Commit message: Update to KiCad 9
Parts:
- moved J1 2.54 mm to (140.4, 49.0)
Other:
- rule pad_to_mask_clearance: 0.2 -> 0.05
